File: imu.kicad_sch (KiCad schematic)
At the start: 3 parts, among them U8 LSM6DSOXTR

Commit message: flash memory module (in a sheet this time)
Pin 1: Chip Select (CS) → PB6 (QUADSPI_BK1_NCS)
Pin 2: IO1 → PC10 (QUADSPI_BK1_IO1)
Pin 3: IO2 → PE2(QUADSPI_BK1_IO2)
Pin 4:  GND → GND
Pin 5: IO0 → PD11(QUADSPI_BK1_IO0)
Pin 6: CLK → PD3(QUADSPI_CLK)
Pin 7: IO3 → PD13(QUADSPI_BK1_IO3)
Pin 8: VSS → VCC (3.3V with decoupling caps)
Connections:
- net SPI1_NSS renamed SPI1_IMU_CS
Changed lines of the file:
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@@
 		)
 	)
-	(label "SPI1_NSS"
+	(label "SPI1_IMU_CS"
 		(at 109.22 77.47 180)
 		(effects
@@
 		)
 	)
-	(embedded_fonts no)
 )
