File: imu.kicad_sch (KiCad schematic)
At the start: 3 parts, among them U8 LSM6DSOXTR

Commit message: Radio (#22)
* MetrocketryRadio

* Fix: moved radio to schematic hierachy

* Cubemx+schematic update

* Screenshots of updates

* Add files via upload

* fix: schematic fix

---------

Co-authored-by: Kisa <kisahassan770@gmail.com>
Co-authored-by: deadman_kisa <74790048+kiki-hassan@users.noreply.github.com>
Connections:
- net GPIO_EXTI0 renamed IMU_ACCEL_EXTI
- net GPIO_EXTI1 renamed IMU_GYRO_EXTI
Changed lines of the file:
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@@
 	(wire
 		(pts
-			(xy 154.94 90.17) (xy 149.86 90.17)
+			(xy 152.4 90.17) (xy 149.86 90.17)
 		)
 		(stroke
@@
 	(wire
 		(pts
-			(xy 154.94 87.63) (xy 149.86 87.63)
+			(xy 152.4 87.63) (xy 149.86 87.63)
 		)
 		(stroke
@@
 		)
 	)
-	(label "GPIO_EXTI1"
-		(at 154.94 90.17 0)
+	(label "IMU_GYRO_EXTI"
+		(at 152.4 90.17 0)
 		(effects
 			(font
@@
 		)
 	)
-	(label "GPIO_EXTI0"
-		(at 154.94 87.63 0)
+	(label "IMU_ACCEL_EXTI"
+		(at 152.4 87.63 0)
 		(effects
 			(font
@@
 		)
 	)
+	(embedded_fonts no)
 )
