File: MetrocketryRadio.kicad_sch (KiCad schematic)
At the start: 12 parts, among them U1 STM32F446VETx, U2 E22-400M30S

Commit message: Add files via upload
new radio
Connections:
- net SPI_MOSI is gone; now on net SPI1_MOSI: U2.17-MOSI
- net Radio_IO0: no longer U2.14-BUSY
- net Radio_IO1: no longer U2.15-NRESET (15-NRST)
- net Radio_IO3: no longer U2.7-TXEN
- net Radio_IO4: no longer U2.6-RXEN
- new net RXEN_Radio: U2.6-RXEN
- new net Radio_BUSY: U2.14-BUSY
- new net Radio_NRST: U2.15-NRESET (15-NRST)
- new net TXEN_Radio: U2.7-TXEN
Changed lines of the file:
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@@
 		)
 	)
-	(label "Radio_IO0"
+	(label "Radio_BUSY"
 		(at 231.14 171.45 0)
 		(effects
@@
 		)
 	)
-	(label "Radio_IO3"
+	(label "TXEN_Radio"
 		(at 280.67 176.53 0)
 		(effects
@@
 		)
 	)
-	(label "Radio_IO1"
+	(label "Radio_NRST"
 		(at 231.14 173.99 0)
 		(effects
@@
 		)
 	)
-	(label "SPI_MOSI"
+	(label "SPI1_MOSI"
 		(at 231.14 179.07 0)
 		(effects
@@
 		)
 	)
-	(label "Radio_IO4"
+	(label "RXEN_Radio"
 		(at 280.67 179.07 0)
 		(effects
