File: 5_pmw_ports.kicad_sch (KiCad schematic)
At the start: 5 parts, among them J1 Conn_01x03, J6 Conn_01x03, J7 Conn_01x03, J8 Conn_01x03, J9 Conn_01x03

Commit message: Changed the pins to use TIM4 and TIM2
Connections:
- net TIM1_CH1_PWM renamed TIM4_CH4
- net TIM2_CH3_PWM renamed TIM4_CH3
- net TIM5_CH4_PWM renamed TIM4_CH1
- net TIM8_CH1_PWM renamed TIM4_CH2
- net TIM9_CH1_PWM renamed TIM2_CH1
Changed lines of the file:
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@@
 		)
 	)
-	(label "TIM9_CH1_PWM"
+	(label "TIM2_CH1"
 		(at 194.31 67.31 180)
 		(effects
@@
 		)
 	)
-	(label "TIM5_CH4_PWM"
+	(label "TIM4_CH1"
 		(at 135.89 69.85 180)
 		(effects
@@
 		)
 	)
-	(label "TIM2_CH3_PWM"
+	(label "TIM4_CH3"
 		(at 102.87 83.82 180)
 		(effects
@@
 		)
 	)
-	(label "TIM8_CH1_PWM"
+	(label "TIM4_CH2"
 		(at 156.21 90.17 180)
 		(effects
@@
 		)
 	)
-	(label "TIM1_CH1_PWM"
+	(label "TIM4_CH4"
 		(at 81.28 68.58 180)
 		(effects
